Commit message: add display flag + tf prefix for turtlebot

File: example/turtlebot3_waffle_pi.urdf.xacro (robot description, xacro)
@@ -1,8 +1,5 @@
 <?xml version="1.0" ?>
-<!-- =================================================================================== -->
-<!-- |    This document was autogenerated by xacro from turtlebot3_waffle_pi.urdf.xacro | -->
-<!-- |    EDITING THIS FILE BY HAND IS NOT RECOMMENDED                                 | -->
-<!-- =================================================================================== -->
-<robot name="turtlebot3_waffle_pi">
+<robot name="turtlebot3_waffle_pi" xmlns:xacro="http://ros.org/wiki/xacro">
+  <xacro:arg name="prefix"    default=""/>
   <!-- Init colour -->
   <material name="black">
@@ -134,5 +131,5 @@
     </plugin>
   </gazebo>
-  <gazebo reference="waffle/base_scan">
+  <gazebo reference="$(arg prefix)base_scan">
     <material>Gazebo/FlatBlack</material>
     <sensor name="lds_lfcd_sensor" type="ray">
@@ -162,5 +159,5 @@
       <plugin filename="libgazebo_ros_laser.so" name="gazebo_ros_lds_lfcd_controller">
         <topicName>scan</topicName>
-        <frameName>waffle/base_scan</frameName>
+        <frameName>$(arg prefix)base_scan</frameName>
       </plugin>
     </sensor>
@@ -187,5 +184,5 @@
         <updateRate>30.0</updateRate>
         <cameraName>camera</cameraName>
-        <frameName>waffle/camera_rgb_optical_frame</frameName>
+        <frameName>$(arg prefix)camera_rgb_optical_frame</frameName>
         <imageTopicName>rgb/image_raw</imageTopicName>
         <cameraInfoTopicName>rgb/camera_info</cameraInfoTopicName>
@@ -199,11 +196,11 @@
     </sensor>
   </gazebo>
-  <link name="waffle/base_footprint"/>
+  <link name="$(arg prefix)base_footprint"/>
   <joint name="base_joint" type="fixed">
-    <parent link="waffle/base_footprint"/>
-    <child link="waffle/base_link"/>
+    <parent link="$(arg prefix)base_footprint"/>
+    <child link="$(arg prefix)base_link"/>
     <origin rpy="0 0 0" xyz="0 0 0.010"/>
   </joint>
-  <link name="waffle/base_link">
+  <link name="$(arg prefix)base_link">
     <visual>
       <origin rpy="0 0 0" xyz="-0.064 0 0.0"/>
@@ -226,10 +223,10 @@
   </link>
   <joint name="wheel_left_joint" type="continuous">
-    <parent link="waffle/base_link"/>
-    <child link="waffle/wheel_left_link"/>
+    <parent link="$(arg prefix)base_link"/>
+    <child link="$(arg prefix)wheel_left_link"/>
     <origin rpy="-1.57 0 0" xyz="0.0 0.144 0.023"/>
     <axis xyz="0 0 1"/>
   </joint>
-  <link name="waffle/wheel_left_link">
+  <link name="$(arg prefix)wheel_left_link">
     <visual>
       <origin rpy="1.57 0 0" xyz="0 0 0"/>
@@ -252,10 +249,10 @@
   </link>
   <joint name="wheel_right_joint" type="continuous">
-    <parent link="waffle/base_link"/>
-    <child link="waffle/wheel_right_link"/>
+    <parent link="$(arg prefix)base_link"/>
+    <child link="$(arg prefix)wheel_right_link"/>
     <origin rpy="-1.57 0 0" xyz="0.0 -0.144 0.023"/>
     <axis xyz="0 0 1"/>
   </joint>
-  <link name="waffle/wheel_right_link">
+  <link name="$(arg prefix)wheel_right_link">
     <visual>
       <origin rpy="1.57 0 0" xyz="0 0 0"/>
@@ -278,9 +275,9 @@
   </link>
   <joint name="caster_back_right_joint" type="fixed">
-    <parent link="waffle/base_link"/>
-    <child link="waffle/caster_back_right_link"/>
+    <parent link="$(arg prefix)base_link"/>
+    <child link="$(arg prefix)caster_back_right_link"/>
     <origin rpy="-1.57 0 0" xyz="-0.177 -0.064 -0.004"/>
   </joint>
-  <link name="waffle/caster_back_right_link">
+  <link name="$(arg prefix)caster_back_right_link">
     <collision>
       <origin rpy="0 0 0" xyz="0 0.001 0"/>
@@ -296,9 +293,9 @@
   </link>
   <joint name="caster_back_left_joint" type="fixed">
-    <parent link="waffle/base_link"/>
-    <child link="waffle/caster_back_left_link"/>
+    <parent link="$(arg prefix)base_link"/>
+    <child link="$(arg prefix)caster_back_left_link"/>
     <origin rpy="-1.57 0 0" xyz="-0.177 0.064 -0.004"/>
   </joint>
-  <link name="waffle/caster_back_left_link">
+  <link name="$(arg prefix)caster_back_left_link">
     <collision>
       <origin rpy="0 0 0" xyz="0 0.001 0"/>
@@ -314,15 +311,15 @@
   </link>
   <joint name="imu_joint" type="fixed">
-    <parent link="waffle/base_link"/>
-    <child link="waffle/imu_link"/>
+    <parent link="$(arg prefix)base_link"/>
+    <child link="$(arg prefix)imu_link"/>
     <origin rpy="0 0 0" xyz="0.0 0 0.068"/>
   </joint>
-  <link name="waffle/imu_link"/>
+  <link name="$(arg prefix)imu_link"/>
   <joint name="scan_joint" type="fixed">
-    <parent link="waffle/base_link"/>
-    <child link="waffle/base_scan"/>
+    <parent link="$(arg prefix)base_link"/>
+    <child link="$(arg prefix)base_scan"/>
     <origin rpy="0 0 0" xyz="-0.064 0 0.122"/>
   </joint>
-  <link name="waffle/base_scan">
+  <link name="$(arg prefix)base_scan">
     <visual>
       <origin rpy="0 0 0" xyz="0 0 0.0"/>
@@ -346,8 +343,8 @@
   <joint name="camera_joint" type="fixed">
     <origin rpy="0 0 0" xyz="0.073 -0.011 0.084"/>
-    <parent link="waffle/base_link"/>
-    <child link="waffle/camera_link"/>
-  </joint>
-  <link name="waffle/camera_link">
+    <parent link="$(arg prefix)base_link"/>
+    <child link="$(arg prefix)camera_link"/>
+  </joint>
+  <link name="$(arg prefix)camera_link">
     <collision>
       <origin rpy="0 0 0" xyz="0.005 0.011 0.013"/>
@@ -359,13 +356,13 @@
   <joint name="camera_rgb_joint" type="fixed">
     <origin rpy="0 0 0" xyz="0.003 0.011 0.009"/>
-    <parent link="waffle/camera_link"/>
-    <child link="waffle/camera_rgb_frame"/>
-  </joint>
-  <link name="waffle/camera_rgb_frame"/>
+    <parent link="$(arg prefix)camera_link"/>
+    <child link="$(arg prefix)camera_rgb_frame"/>
+  </joint>
+  <link name="$(arg prefix)camera_rgb_frame"/>
   <joint name="camera_rgb_optical_joint" type="fixed">
     <origin rpy="-1.57 0 -1.57" xyz="0 0 0"/>
-    <parent link="waffle/camera_rgb_frame"/>
-    <child link="waffle/camera_rgb_optical_frame"/>
-  </joint>
-  <link name="waffle/camera_rgb_optical_frame"/>
+    <parent link="$(arg prefix)camera_rgb_frame"/>
+    <child link="$(arg prefix)camera_rgb_optical_frame"/>
+  </joint>
+  <link name="$(arg prefix)camera_rgb_optical_frame"/>
 </robot>
